File: pcb/light-bar/light-bar.sch (KiCad schematic (older format))
At the start: 21 parts

Commit message: Moved mounting holes
Parts:
- D1, D10, D2, D3, D4, D5, D6, D7, D8, D9: symbol Device:LED_Small -> light-bar-rescue:LED_Small-Device
- J?: symbol Connector_Generic:Conn_01x02 -> light-bar-rescue:Conn_01x02-Connector_Generic
- R1, R10, R2, R3, R4, R5, R6, R7, R8, R9: symbol Device:R_Small -> light-bar-rescue:R_Small-Device
Changed lines of the file:
@@
 $EndDescr
 $Comp
-L power:VCC #PWR0102
+L light-bar-rescue:VCC-power #PWR0102
 U 1 1 5F7FEF21
 P 750 1550
@@
 $EndComp
 $Comp
-L Device:LED_Small D1
+L light-bar-rescue:LED_Small-Device D1
 U 1 1 5F7FF59B
 P 900 1450
@@
 $EndComp
 $Comp
-L Device:R_Small R1
+L light-bar-rescue:R_Small-Device R1
 U 1 1 5F80069B
 P 900 1150
@@
 	900  1250 900  1350
 $Comp
-L Device:LED_Small D2
+L light-bar-rescue:LED_Small-Device D2
 U 1 1 5F80428F
 P 1450 1450
@@
 $EndComp
 $Comp
-L Device:R_Small R2
+L light-bar-rescue:R_Small-Device R2
 U 1 1 5F804295
 P 1450 1150
@@
 	1450 1250 1450 1350
 $Comp
-L Device:LED_Small D3
+L light-bar-rescue:LED_Small-Device D3
 U 1 1 5F80547C
 P 2000 1450
@@
 $EndComp
 $Comp
-L Device:R_Small R3
+L light-bar-rescue:R_Small-Device R3
 U 1 1 5F805482
 P 2000 1150
@@
 	2000 1250 2000 1350
 $Comp
-L Device:LED_Small D4
+L light-bar-rescue:LED_Small-Device D4
 U 1 1 5F80B2EA
 P 2550 1450
@@
 $EndComp
 $Comp
-L Device:R_Small R4
+L light-bar-rescue:R_Small-Device R4
 U 1 1 5F80B2F0
 P 2550 1150
@@
 	2550 1250 2550 1350
 $Comp
-L Device:LED_Small D5
+L light-bar-rescue:LED_Small-Device D5
 U 1 1 5F80B2F7
 P 3100 1450
@@
 $EndComp
 $Comp
-L Device:R_Small R5
+L light-bar-rescue:R_Small-Device R5
 U 1 1 5F80B2FD
 P 3100 1150
@@
 	3100 1250 3100 1350
 $Comp
-L Device:LED_Small D6
+L light-bar-rescue:LED_Small-Device D6
 U 1 1 5F80B304
 P 3650 1450
@@
 $EndComp
 $Comp
-L Device:R_Small R6
+L light-bar-rescue:R_Small-Device R6
 U 1 1 5F80B30A
 P 3650 1150
@@
 	3650 1250 3650 1350
 $Comp
-L Device:LED_Small D7
+L light-bar-rescue:LED_Small-Device D7
 U 1 1 5F81057A
 P 4200 1450
@@
 $EndComp
 $Comp
-L Device:R_Small R7
+L light-bar-rescue:R_Small-Device R7
 U 1 1 5F810580
 P 4200 1150
@@
 	4200 1250 4200 1350
 $Comp
-L Device:LED_Small D8
+L light-bar-rescue:LED_Small-Device D8
 U 1 1 5F810587
 P 4750 1450
@@
 $EndComp
 $Comp
-L Device:R_Small R8
+L light-bar-rescue:R_Small-Device R8
 U 1 1 5F81058D
 P 4750 1150
@@
 	4750 1250 4750 1350
 $Comp
-L Device:LED_Small D9
+L light-bar-rescue:LED_Small-Device D9
 U 1 1 5F810594
 P 5300 1450
@@
 $EndComp
 $Comp
-L Device:R_Small R9
+L light-bar-rescue:R_Small-Device R9
 U 1 1 5F81059A
 P 5300 1150
@@
 	5300 1250 5300 1350
 $Comp
-L Device:LED_Small D10
+L light-bar-rescue:LED_Small-Device D10
 U 1 1 5F8105A1
 P 5850 1450
@@
 $EndComp
 $Comp
-L Device:R_Small R10
+L light-bar-rescue:R_Small-Device R10
 U 1 1 5F8105A7
 P 5850 1150
@@
 	750  1050 900  1050
 $Comp
-L power:GND #PWR0101
+L light-bar-rescue:GND-power #PWR0101
 U 1 1 5F7FE936
 P 750 1050
@@
 $EndComp
 $Comp
-L Connector_Generic:Conn_01x02 J?
+L light-bar-rescue:Conn_01x02-Connector_Generic J?
 U 1 1 5F84685C
 P 900 1750
